File: HW/NANO5/Nano5/Nano5.kicad_sch (KiCad schematic)
At the start: 131 parts, among them J1 Screw_Terminal_01x03, J10 Screw_Terminal_01x03, J11 Screw_Terminal_01x03, J12 Screw_Terminal_01x02, J13 Conn_02x04_Counter_Clockwise, J14 Conn_02x04_Counter_Clockwise, J15 Conn_02x03_Counter_Clockwise, J16 Conn_01x02, J17 Conn_01x02, J2 Screw_Terminal_01x03, J3 Screw_Terminal_01x03, J4 Screw_Terminal_01x03, J5 Screw_Terminal_01x02, J6 Screw_Terminal_01x02, J7 Screw_Terminal_01x02, J8 Screw_Terminal_01x03, J9 Screw_Terminal_01x03, K1 SANYOU_SRD_Form_C, K2 SANYOU_SRD_Form_C, K3 SANYOU_SRD_Form_C, K4 SANYOU_SRD_Form_C, K5 SANYOU_SRD_Form_C, K6 SANYOU_SRD_Form_C, Q1 MMBT3904, Q2 MMBT3904, Q3 MMBT3904, Q4 MMBT3904, Q5 MMBT3904, Q6 MMBT3904, U1 ATmega328P-A, U10 ESP-12E, U11 M24C02-RMN, U12 ST485EBDR, U13 DS1307Z+, U14 MP1584, U15 LM358, U16 AP1117-33, U2 LTV-817S, U3 LTV-817S, U4 LTV-817S, U5 LTV-817S, U6 LTV-817S, U7 LTV-817S, U8 LTV-817S, U9 LTV-817S, Y1 Crystal_Small

Commit message: MAJOR UPDATE
Parts:
- added BT2: Battery_Cell, Battery:BatteryHolder_Keystone_1058_1x2032, symbol Device:Battery_Cell
- added C19, C20: C_Small, Capacitor_SMD:C_0805_2012Metric, symbol Device:C_Small
- added C21, C22, C23, C24: 100nF, Capacitor_SMD:C_0805_2012Metric, symbol Device:C_Small
- added C25: C_Polarized_Small, Capacitor_SMD:CP_Elec_4x3.9, symbol Device:C_Polarized_Small
- added J18: Conn_01x05, Connector_PinHeader_2.54mm:PinHeader_1x05_P2.54mm_Vertical, symbol Connector_Generic:Conn_01x05
- added JP1: Jumper_2_Open, Jumper:SolderJumper-2_P1.3mm_Open_RoundedPad1.0x1.5mm, symbol Jumper:Jumper_2_Open
- added JP2, JP3, JP4: Jumper_2_Open, Jumper:SolderJumper-2_P1.3mm_Bridged_RoundedPad1.0x1.5mm, symbol Jumper:Jumper_2_Open
- added Q10, Q7, Q8, Q9: MMBT3904, Package_TO_SOT_SMD:SOT-23, symbol Transistor_BJT:MMBT3904
- added R39, R40, R41, R42, R43, R44, R45, R46, R47, R48, R49, R50, R51, R52, R53, R54, R55, R56, R57, R58, R59: R, Resistor_SMD:R_0805_2012Metric, symbol Device:R
- added SW1: SW_DIP_x02, Button_Switch_SMD:SW_DIP_SPSTx02_Slide_6.7x6.64mm_W8.61mm_P2.54mm_LowProfile, symbol Switch:SW_DIP_x02
- added Y2: Crystal_GND3_Small, Crystal:Crystal_SMD_FrontierElectronics_FM206, symbol Device:Crystal_GND3_Small
Connections:
- net +3V3: now also U16.2 (VO), R52.1, R53.1, R54.1, R55.1, R57.1, R58.1
- net +5V: now also D23.2, D24.2, U14.4 (+VOUT), U16.3 (VI), C25.1, JP2.2 (B), JP3.2 (B), JP4.2 (B), R42.1, R50.1, R51.1, R56.1
- net A0: now also U2.4; no longer U3.4
- net A1: now also U3.4; no longer U4.4
- net A2: now also U4.4; no longer U5.4
- net A3: now also U5.4
- net A6: now also C19.1
- net A7: now also C20.1
- net D10: no longer U8.4
- net D11: now also R3.2; no longer U7.4
- net D12: now also R2.2; no longer U6.4
- net D13: now also R1.2; no longer U2.4
- net D2: now also U6.4; no longer U9.4
- net D3: now also U7.4; no longer R1.2
- net D4: now also U8.4; no longer R2.2
- net D5: now also U9.4; no longer R3.2
- net D9: now also R39.2
- net ED1: now also Q8.2 (E), R54.2
- net ED2: now also Q9.2 (E), R55.2
- net GND: now also D23.1, D24.1, U11.1 (E0), U11.2 (E1), U11.3 (E2), U11.4 (VSS), U11.7 (~{WC}), U12.4 (DI), U12.5 (GND), U13.4 (GND), U14.3 (-VOUT), U15.4 (V-), U16.1 (GND), BT2.2 (-), C19.2, C20.2, C21.1, C22.1, C23.1, C24.1, C25.2, Q7.2 (E), R40.2, R43.2, R47.2
- net RXE: now also Q10.2 (E), R58.2
- net TXE: now also SW1.4
- net X1: now also Y1.1; no longer Y1.2
- net X2: now also Y1.2; no longer Y1.1
- net at J15.5 (Pin_5): no longer R29.2
- net RO: now reaches U12.1 (RO)
- net RO: now also SW1.3
- net at U12.2 (~{RE}): now also U12.3 (DE), Q7.3 (C), R42.2
- net at U12.6 (A): now also R46.1, R48.2, R49.2
- net at U12.7 (B): now also JP1.1 (A), R45.1, R47.1
- net at U12.8 (VCC): now also JP4.1 (A), R49.1
- net VIN: now reaches C18.2, F1.1, U14.2 (+VIN)
- net VIN: now also U15.8 (V+), C24.2
- net at U15.1: now also U15.2 (-), U15.5 (+)
- net at U15.3 (+): now also C22.2, R39.1, R40.1
- net at J15.4 (Pin_4): no longer R30.2
- net at U15.6 (-): now also R43.1, R44.1
- net at U15.7: now also R44.2, R59.1
- net at U13.1 (X1): now also Y2.1
- net at U13.2 (X2): now also Y2.2
- net at U13.3 (VBAT): now also BT2.1 (+)
- net at U13.8 (VCC): now also C23.2, JP3.1 (A)
- net at U11.8 (VCC): now also JP2.1 (A)
- net at U1.20 (AREF): now also C21.2
- new net: Q9.1 (B), R53.2
- new net: Q9.3 (C), R51.2
- new net: Q10.1 (B), R57.2
- new net: JP1.2 (B), R48.1
- new net: Q7.1 (B), R41.1
- new net: Q8.1 (B), R52.2
- new net: Q8.3 (C), R50.2
- new net RD0: R29.2, SW1.1, SW1.2
- new net XD1: Q10.3 (C), R30.2, R41.2, R56.2
Other:
- moved on the sheet: C17, C18, D21, D22, D23, D24, F1, H1, J12, J13, J15, J16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

Commit message: major update
Connections:
- net A4: now also Q9.3 (C), R51.2
- net A5: now also Q8.3 (C), R50.2
Changed lines of the file:
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@@
+    )
+  )
+  (global_label "A5" (shape input) (at 327.66 181.61 180) (fields_autoplaced)
+    (effects (font (size 1.27 1.27)) (justify right))
+    (property "Intersheet References" "${INTERSHEET_REFS}" (id 0) (at 322.9488 181.6894 0)
+      (effects (font (size 1.27 1.27)) (justify right) hide)
     )
   )
@@
     )
   )
+  (global_label "A4" (shape input) (at 327.66 196.85 180) (fields_autoplaced)
+    (effects (font (size 1.27 1.27)) (justify right))
+    (property "Intersheet References" "${INTERSHEET_REFS}" (id 0) (at 322.9488 196.9294 0)
+      (effects (font (size 1.27 1.27)) (justify right) hide)
+    )
+  )

Commit message: update 2104
Parts:
- added D25: LED, LED_SMD:LED_0805_2012Metric, symbol Device:LED
- added R60: R, Resistor_SMD:R_0805_2012Metric, symbol Device:R
- added SW2, SW3: SW_Push, Button_Switch_SMD:SW_SPST_B3U-1000P, symbol Switch:SW_Push
Connections:
- net +5V: now also R60.2
- net ED0: now also J18.5 (Pin_5)
- net ERST: now also J18.4 (Pin_4), SW2.1
- net GND: now also J18.1 (Pin_1), J6.1 (Pin_1), D25.1 (K), SW2.2, SW3.2
- net RST: now also SW3.1
- net RXE: now also J18.2 (Pin_2)
- net TXE: now also J18.3 (Pin_3)
- net AO: now reaches J6.2 (Pin_2)
- net AO: now also R59.2
- net OA: now reaches J5.1 (Pin_1)
- net OA: now also R46.2
- net OB: now reaches J5.2 (Pin_2)
- net OB: now also R45.2
- net at J17.1 (Pin_1), R32.2, R34.2: now also J8.3 (Pin_3); no longer J8.1 (Pin_1)
- net at J16.1 (Pin_1), R31.2, R33.1: now also J8.1 (Pin_1); no longer J8.3 (Pin_3)
- new net: D25.2 (A), R60.1
Other:
- moved on the sheet: J18, J5, J6, J7

Commit message: fix update
Parts:
- added L1: L_Ferrite_Small, Inductor_SMD:L_1806_4516Metric_Pad1.45x1.90mm_HandSolder, symbol Device:L_Ferrite_Small
- F1: footprint Fuse:Fuse_0805_2012Metric -> Fuse:Fuse_1812_4532Metric
Connections:
- net +3V3: now also J13.2 (Pin_2), J14.2 (Pin_2)
- net +5V: now also J13.1 (Pin_1), J14.1 (Pin_1)
- net A4: now also J13.4 (Pin_4), J14.6 (Pin_6)
- net A5: now also J13.6 (Pin_6), J14.4 (Pin_4)
- net GND: now also J13.7 (Pin_7), J13.8 (Pin_8), J14.7 (Pin_7), J14.8 (Pin_8), U14.1 (-VIN)
- net OA: now also J13.5 (Pin_5), J14.5 (Pin_5)
- net OB: now also J13.3 (Pin_3), J14.3 (Pin_3)
- net at K3.1: now also J2.2 (Pin_2)
- net at K3.3: now also J2.1 (Pin_1)
- net at K5.1: now also J3.1 (Pin_1)
- net at K5.3: now also J4.3 (Pin_3)
- net at K1.1: now also J1.3 (Pin_3)
- net at K1.3: now also J1.2 (Pin_2)
- net at F1.2: now also L1.2; no longer D22.1 (K)
- net at J2.3 (Pin_3): now also K2.3
- net at J3.2 (Pin_2): now also K4.3
- net at J3.3 (Pin_3): now also K4.1
- net at K6.1: now also J4.2 (Pin_2)
- net at K6.3: now also J4.1 (Pin_1)
- net at J1.1 (Pin_1): now also K2.1
- new net: D22.1 (K), L1.1
Other:
- moved on the sheet: C18, C25, D22, F1, J12, J3, J4, U14, U16

Commit message: ISP
Parts:
- added JP5, JP6, JP7: SolderJumper_3_Open, Jumper:SolderJumper-3_P1.3mm_Open_RoundedPad1.0x1.5mm, symbol Jumper:SolderJumper_3_Open
Connections:
- net +5V: now also J15.2 (Pin_2)
- net D11: now also J15.4 (Pin_4)
- net D12: now also JP6.3 (B)
- net D13: now also JP7.3 (B)
- net GND: now also J15.6 (Pin_6)
- net RD0: now also JP6.1 (A)
- net RST: now also JP5.3 (B)
- net XD1: now also JP7.1 (A)
- net DTR: now reaches C17.1
- net DTR: now also JP5.1 (A)
- net JD12: now reaches J15.1 (Pin_1)
- net JD12: now also JP6.2 (C)
- net JD13: now reaches J15.3 (Pin_3)
- net JD13: now also JP7.2 (C)
- net JRST: now reaches J15.5 (Pin_5)
- net JRST: now also JP5.2 (C)

Commit message: fix track
Parts:
- added JP8: Jumper_2_Bridged, Jumper:SolderJumper-2_P1.3mm_Bridged2Bar_RoundedPad1.0x1.5mm, symbol Jumper:Jumper_2_Bridged
- added TP1: TestPoint, TestPoint:TestPoint_Pad_D1.0mm, symbol Connector:TestPoint
- JP2, JP3, JP4: footprint Jumper:SolderJumper-2_P1.3mm_Bridged_RoundedPad1.0x1.5mm -> Jumper:SolderJumper-2_P1.3mm_Open_RoundedPad1.0x1.5mm
Connections:
- net +5V: now also J7.1 (Pin_1), JP8.1 (A)
- net D10: now also TP1.1
- net GND: now also J12.2 (Pin_2), J7.2 (Pin_2)
- net +5P: now reaches D2.1 (K), K2.2, R8.2
- net +5P: now also D1.1 (K), D3.1 (K), D4.1 (K), D5.1 (K), D6.1 (K), K1.2, K3.2, K4.2, K5.2, K6.2, R10.2, R11.2, R12.2, R7.2, R9.2, JP8.2 (B)

Commit message: update annote
Parts:
- removed H1, H2, H3, H4: MountingHole, MountingHole:MountingHole_3.2mm_M3, symbol Mechanical:MountingHole
- added FID1, FID2, FID3, FID4: Fiducial, Fiducial:Fiducial_1.5mm_Mask3mm, symbol Mechanical:Fiducial
- added H1, H2, H3, H4: MountingHole_Pad, MountingHole:MountingHole_3.2mm_M3_Pad_Via, symbol Mechanical:MountingHole_Pad
- added JP9: Jumper_2_Bridged, Jumper:SolderJumper-2_P1.3mm_Bridged_RoundedPad1.0x1.5mm, symbol Jumper:Jumper_2_Bridged
- added Re1: R, Resistor_THT:R_Axial_DIN0207_L6.3mm_D2.5mm_P10.16mm_Horizontal, symbol Device:R
Connections:
- net +5V: now also J7.2 (Pin_2); no longer J7.1 (Pin_1)
- net GND: now also J7.1 (Pin_1), J8.2 (Pin_2), Re1.2; no longer J7.2 (Pin_2)
- net RXE: now also JP9.2 (B); no longer Q10.2 (E), R58.2
- new net: H3.1, Re1.1
- new net: JP9.1 (A), Q10.2 (E), R58.2
