File: HW/NANO5/Nano5/_autosave-Nano5.kicad_pcb (KiCad board)
At the start: 2 copper layers, 100 x 90 mm, 134 parts, among them J1 Screw_Terminal_01x03, J10 Screw_Terminal_01x03, J11 Screw_Terminal_01x03, J12 Screw_Terminal_01x02, J13 Conn_02x04_Counter_Clockwise, J14 Conn_02x04_Counter_Clockwise, J15 Conn_02x03_Counter_Clockwise, J16 Conn_01x02, J17 Conn_01x02, J2 Screw_Terminal_01x03, J3 Screw_Terminal_01x03, J4 Screw_Terminal_01x03, J5 Screw_Terminal_01x02, J6 Screw_Terminal_01x02, J7 Screw_Terminal_01x02, J8 Screw_Terminal_01x03, J9 Screw_Terminal_01x03, K1 SANYOU_SRD_Form_C, K2 SANYOU_SRD_Form_C, K3 SANYOU_SRD_Form_C, K4 SANYOU_SRD_Form_C, K5 SANYOU_SRD_Form_C, K6 SANYOU_SRD_Form_C, Q1 MMBT3904, Q2 MMBT3904, Q3 MMBT3904, Q4 MMBT3904, Q5 MMBT3904, Q6 MMBT3904, U1 ATmega328P-A, U10 ESP-12E, U11 M24C02-RMN, U12 ST485EBDR, U13 DS1307Z+, U14 MP1584, U15 LM358, U16 AP1117-33, U2 LTV-817S, U3 LTV-817S, U4 LTV-817S, U5 LTV-817S, U6 LTV-817S, U7 LTV-817S, U8 LTV-817S, U9 LTV-817S, Y1 Crystal_Small

Commit message: update
Routing:
- net Net-(U1-Pad20): track 0.25 -> 6.62 mm, vias 0 -> 2
- net +5V: track 23.5 -> 29.7 mm
Changed lines of the file:
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@@
   (via (at 101.4765 75.248912) (size 0.6) (drill 0.3) (layers "F.Cu" "B.Cu") (net 168))
   (via (at 94.7 85.95) (size 0.6) (drill 0.3) (layers "F.Cu" "B.Cu") (net 168))
-  (segment (start 101.4765 75.248912) (end 101.4765 76.1735) (width 0.2) (layer "B.Cu") (net 168))
-  (segment (start 101.4765 76.1735) (end 94.7 82.95) (width 0.2) (layer "B.Cu") (net 168))
-  (segment (start 94.7 82.95) (end 94.7 85.95) (width 0.2) (layer "B.Cu") (net 168))
+  (segment (start 101.4765 75.248912) (end 101.4765 76.0235) (width 0.2) (layer "B.Cu") (net 168))
+  (segment (start 101.4765 76.0235) (end 94.7 82.8) (width 0.2) (layer "B.Cu") (net 168))
+  (segment (start 94.7 82.8) (end 94.7 85.95) (width 0.2) (layer "B.Cu") (net 168))
   (segment (start 139.275 70.55) (end 103.45 70.55) (width 0.2) (layer "F.Cu") (net 169))
   (segment (start 147.625 68.05) (end 146.175 69.5) (width 0.2) (layer "F.Cu") (net 169))
@@
   (segment (start 104.175 80.9) (end 102.895 79.62) (width 0.2) (layer "F.Cu") (net 175))
   (segment (start 111.97 81.91) (end 112.89 80.99) (width 0.2) (layer "F.Cu") (net 175))
-  (segment (start 100.15 81.375) (end 101.14 81.375) (width 0.4) (layer "F.Cu") (net 175))
+  (segment (start 100.15 81.375) (end 101.14 81.375) (width 0.2) (layer "F.Cu") (net 175))
   (segment (start 105.6 80.9) (end 104.175 80.9) (width 0.2) (layer "F.Cu") (net 175))
   (segment (start 107.7425 81.91) (end 106.61 81.91) (width 0.2) (layer "F.Cu") (net 175))
   (segment (start 107.7425 81.91) (end 111.97 81.91) (width 0.2) (layer "F.Cu") (net 175))
-  (segment (start 101.14 81.375) (end 102.895 79.62) (width 0.4) (layer "F.Cu") (net 175))
-  (segment (start 101.43 78.975) (end 102.895 77.51) (width 0.4) (layer "F.Cu") (net 176))
+  (segment (start 101.14 81.375) (end 102.895 79.62) (width 0.2) (layer "F.Cu") (net 175))
+  (segment (start 101.43 78.975) (end 102.895 77.51) (width 0.2) (layer "F.Cu") (net 176))
   (segment (start 107.6625 78.22) (end 111.93 78.22) (width 0.2) (layer "F.Cu") (net 176))
   (segment (start 106.53 78.22) (end 106.1 78.65) (width 0.2) (layer "F.Cu") (net 176))
@@
   (segment (start 111.93 78.22) (end 112.88 77.27) (width 0.2) (layer "F.Cu") (net 176))
   (segment (start 104.035 78.65) (end 102.895 77.51) (width 0.2) (layer "F.Cu") (net 176))
-  (segment (start 100.15 78.975) (end 101.43 78.975) (width 0.4) (layer "F.Cu") (net 176))
+  (segment (start 100.15 78.975) (end 101.43 78.975) (width 0.2) (layer "F.Cu") (net 176))
   (segment (start 88.646 90.221) (end 88.625 90.2) (width 0.2) (layer "F.Cu") (net 177))
   (segment (start 88.646 90.231) (end 88.646 90.221) (width 0.2) (layer "F.Cu") (net 177))
@@
   (segment (start 91.65 81.375) (end 88.55 81.375) (width 0.4) (layer "F.Cu") (net 190))
   (segment (start 98.475 82.175) (end 96.925 80.625) (width 0.4) (layer "F.Cu") (net 190))
+  (segment (start 107.28 86.37) (end 103.42 86.37) (width 0.4) (layer "F.Cu") (net 190))
   (segment (start 93.125 80) (end 92.9 79.775) (width 0.4) (layer "F.Cu") (net 190))
   (segment (start 94.075 71.2) (end 98.55 71.2) (width 0.2) (layer "F.Cu") (net 190))
@@
   (segment (start 93.125 81.15) (end 93.125 80.625) (width 0.4) (layer "F.Cu") (net 190))
   (segment (start 100.15 82.175) (end 100.945 82.175) (width 0.4) (layer "F.Cu") (net 190))
+  (segment (start 102.83 85.78) (end 102.83 84.26) (width 0.4) (layer "F.Cu") (net 190))
   (segment (start 100.945 82.175) (end 102.91 84.14) (width 0.4) (layer "F.Cu") (net 190))
+  (segment (start 103.42 86.37) (end 102.83 85.78) (width 0.4) (layer "F.Cu") (net 190))
   (segment (start 86.77 111.705) (end 89.425 109.05) (width 0.2) (layer "F.Cu") (net 191))
   (segment (start 86.77 114.33) (end 86.77 111.705) (width 0.2) (layer "F.Cu") (net 191))
@@
   (segment (start 102.825 82.175) (end 102.85 82.15) (width 0.4) (layer "F.Cu") (net 201))
   (segment (start 102.9 82.2) (end 102.875 82.175) (width 0.4) (layer "F.Cu") (net 201))
+  (segment (start 100.15 80.575) (end 99.175 80.575) (width 0.2) (layer "F.Cu") (net 201))
+  (segment (start 99.175 80.575) (end 98.625 81.125) (width 0.2) (layer "F.Cu") (net 201))
   (segment (start 102.9 82.2) (end 102.85 82.15) (width 0.4) (layer "F.Cu") (net 201))
+  (via (at 98.625 81.125) (size 0.6) (drill 0.3) (layers "F.Cu" "B.Cu") (net 201))
+  (via (at 102.85 82.075) (size 0.6) (drill 0.3) (layers "F.Cu" "B.Cu") (net 201))
+  (segment (start 99.575 82.075) (end 102.85 82.075) (width 0.2) (layer "B.Cu") (net 201))
+  (segment (start 98.625 81.125) (end 99.575 82.075) (width 0.2) (layer "B.Cu") (net 201))
   (zone (net 85) (net_name "GNDA") (layer "F.Cu") (hatch edge 0.508)
     (connect_pads thru_hole_only (clearance 0.508))
@@
       (pts
         (xy 127.975 97.45)
-        (xy 127.975 102)
-        (xy 125.825 104.15)
+        (xy 127.975 100.625)
+        (xy 125.775 102.425)
         (xy 125.725 120.225)
         (xy 78.618343 120.200311)
