File: HW/NANO5/Nano5/_autosave-Nano5.kicad_sch (KiCad schematic)
At the start: 131 parts, among them J1 Screw_Terminal_01x03, J10 Screw_Terminal_01x03, J11 Screw_Terminal_01x03, J12 Screw_Terminal_01x02, J13 Conn_02x04_Counter_Clockwise, J14 Conn_02x04_Counter_Clockwise, J15 Conn_02x03_Counter_Clockwise, J16 Conn_01x02, J17 Conn_01x02, J2 Screw_Terminal_01x03, J3 Screw_Terminal_01x03, J4 Screw_Terminal_01x03, J5 Screw_Terminal_01x02, J6 Screw_Terminal_01x02, J7 Screw_Terminal_01x02, J8 Screw_Terminal_01x03, J9 Screw_Terminal_01x03, K1 SANYOU_SRD_Form_C, K2 SANYOU_SRD_Form_C, K3 SANYOU_SRD_Form_C, K4 SANYOU_SRD_Form_C, K5 SANYOU_SRD_Form_C, K6 SANYOU_SRD_Form_C, Q1 MMBT3904, Q2 MMBT3904, Q3 MMBT3904, Q4 MMBT3904, Q5 MMBT3904, Q6 MMBT3904, U1 ATmega328P-A, U10 ESP-12E, U11 M24C02-RMN, U12 ST485EBDR, U13 DS1307Z+, U14 MP1584, U15 LM358, U16 AP1117-33, U2 LTV-817S, U3 LTV-817S, U4 LTV-817S, U5 LTV-817S, U6 LTV-817S, U7 LTV-817S, U8 LTV-817S, U9 LTV-817S, Y1 Crystal_Small

Commit message: update
Parts:
- added C19, C20: C_Small, Capacitor_SMD:C_0805_2012Metric, symbol Device:C_Small
- added C21: 100nF, Capacitor_SMD:C_0805_2012Metric, symbol Device:C_Small
Connections:
- net A6: now also C19.1
- net A7: now also C20.1
- net GND: now also D23.1, D24.1, C19.2, C20.2, C21.1
- net at U14.4 (+VOUT): now also U16.3 (VI)
- net at U1.20 (AREF): now also C21.2
Other:
- moved on the sheet: C18, D22, F1, J12, U14, U16
