File: HW/NANO5/Nano5/Nano5.kicad_pcb (KiCad board)
At the start: 2 copper layers, 100 x 90 mm, 134 parts, among them J1 Screw_Terminal_01x03, J10 Screw_Terminal_01x03, J11 Screw_Terminal_01x03, J12 Screw_Terminal_01x02, J13 Conn_02x04_Counter_Clockwise, J14 Conn_02x04_Counter_Clockwise, J15 Conn_02x03_Counter_Clockwise, J16 Conn_01x02, J17 Conn_01x02, J2 Screw_Terminal_01x03, J3 Screw_Terminal_01x03, J4 Screw_Terminal_01x03, J5 Screw_Terminal_01x02, J6 Screw_Terminal_01x02, J7 Screw_Terminal_01x02, J8 Screw_Terminal_01x03, J9 Screw_Terminal_01x03, K1 SANYOU_SRD_Form_C, K2 SANYOU_SRD_Form_C, K3 SANYOU_SRD_Form_C, K4 SANYOU_SRD_Form_C, K5 SANYOU_SRD_Form_C, K6 SANYOU_SRD_Form_C, Q1 MMBT3904, Q2 MMBT3904, Q3 MMBT3904, Q4 MMBT3904, Q5 MMBT3904, Q6 MMBT3904, U1 ATmega328P-A, U10 ESP-12E, U11 M24C02-RMN, U12 ST485EBDR, U13 DS1307Z+, U14 MP1584, U15 LM358, U16 AP1117-33, U2 LTV-817S, U3 LTV-817S, U4 LTV-817S, U5 LTV-817S, U6 LTV-817S, U7 LTV-817S, U8 LTV-817S, U9 LTV-817S, Y1 Crystal_Small

Commit message: MAJOR UPDATE
Parts:
- added BT2: Battery_Cell, Battery:BatteryHolder_Keystone_1058_1x2032, B.Cu at (136.5, 81.0)
- added C22: 100nF, Capacitor_SMD:C_0805_2012Metric, F.Cu at (125.3, 73.2)
- added C23: 100nF, Capacitor_SMD:C_0805_2012Metric, F.Cu at (112.3, 82.7)
- added C24: 100nF, Capacitor_SMD:C_0805_2012Metric, F.Cu at (137.7, 72.0)
- added C25: C_Polarized_Small, Capacitor_SMD:CP_Elec_4x3.9, F.Cu at (141.7, 87.6)
- added J18: Conn_01x05, Connector_PinHeader_2.54mm:PinHeader_1x05_P2.54mm_Vertical, F.Cu at (143.8, 68.7)
- added JP1: Jumper_2_Open, Jumper:SolderJumper-2_P1.3mm_Open_RoundedPad1.0x1.5mm, F.Cu at (121.0, 74.0)
- added JP2: Jumper_2_Open, Jumper:SolderJumper-2_P1.3mm_Bridged_RoundedPad1.0x1.5mm, B.Cu at (105.7, 84.3)
- added JP3: Jumper_2_Open, Jumper:SolderJumper-2_P1.3mm_Bridged_RoundedPad1.0x1.5mm, B.Cu at (112.3, 84.3)
- added JP4: Jumper_2_Open, Jumper:SolderJumper-2_P1.3mm_Bridged_RoundedPad1.0x1.5mm, B.Cu at (114.6, 70.9)
- added Q10: MMBT3904, Package_TO_SOT_SMD:SOT-23, F.Cu at (141.2, 79.8)
- added Q7: MMBT3904, Package_TO_SOT_SMD:SOT-23, F.Cu at (107.1, 73.7)
- added Q8: MMBT3904, Package_TO_SOT_SMD:SOT-23, F.Cu at (153.9, 99.2)
- added Q9: MMBT3904, Package_TO_SOT_SMD:SOT-23, F.Cu at (149.8, 99.1)
- added R39: R, Resistor_SMD:R_0805_2012Metric, F.Cu at (125.3, 77.5)
- added R40: R, Resistor_SMD:R_0805_2012Metric, F.Cu at (125.3, 75.4)
- added R41: R, Resistor_SMD:R_0805_2012Metric, F.Cu at (101.8, 73.6)
- added R42: R, Resistor_SMD:R_0805_2012Metric, F.Cu at (104.0, 73.6)
- added R43: R, Resistor_SMD:R_0805_2012Metric, F.Cu at (133.0, 77.5)
- added R44: R, Resistor_SMD:R_0805_2012Metric, F.Cu at (136.9, 74.7)
- added R45: R, Resistor_SMD:R_0805_2012Metric, F.Cu at (118.0, 70.9)
- added R46: R, Resistor_SMD:R_0805_2012Metric, F.Cu at (119.3, 76.8)
- added R47: R, Resistor_SMD:R_0805_2012Metric, F.Cu at (121.6, 70.9)
- added R48: R, Resistor_SMD:R_0805_2012Metric, F.Cu at (118.5, 74.0)
- added R49: R, Resistor_SMD:R_0805_2012Metric, F.Cu at (114.4, 70.9)
- added R50: R, Resistor_SMD:R_0805_2012Metric, F.Cu at (152.9, 94.8)
- added R51: R, Resistor_SMD:R_0805_2012Metric, F.Cu at (145.9, 101.6)
- added R52: R, Resistor_SMD:R_0805_2012Metric, F.Cu at (150.9, 94.8)
- added R53: R, Resistor_SMD:R_0805_2012Metric, F.Cu at (148.9, 94.8)
- added R54: R, Resistor_SMD:R_0805_2012Metric, F.Cu at (154.9, 91.3)
- added R55: R, Resistor_SMD:R_0805_2012Metric, F.Cu at (157.8, 90.6)
- added R56: R, Resistor_SMD:R_0805_2012Metric, F.Cu at (138.2, 85.4)
- added R57: R, Resistor_SMD:R_0805_2012Metric, F.Cu at (142.3, 75.9)
- added R58: R, Resistor_SMD:R_0805_2012Metric, F.Cu at (140.2, 75.9)
- added R59: R, Resistor_SMD:R_0805_2012Metric, F.Cu at (125.3, 71.2)
- added SW1: SW_DIP_x02, Button_Switch_SMD:SW_DIP_SPSTx02_Slide_6.7x6.64mm_W8.61mm_P2.54mm_LowProfile, F.Cu at (128.4, 82.4)
- added Y2: Crystal_GND3_Small, Crystal:Crystal_SMD_FrontierElectronics_FM206, F.Cu at (116.6, 86.6)
- moved R32 41.1 mm to (136.3, 102.7), turned to -90 degrees
- moved R31 38.1 mm to (134.2, 102.7), turned to -90 degrees
- moved D23 29.7 mm to (137.4, 89.4), turned to 90 degrees
- moved D24 25.8 mm to (131.8, 89.4), turned to 90 degrees
- moved C19 22.9 mm to (134.6, 89.2)
- moved U11 22.2 mm to (106.4, 83.6), turned to 180 degrees
- moved C20 19.5 mm to (129.0, 89.2)
- moved C17 17.3 mm to (75.9, 70.1)
- moved C21 17.3 mm to (87.6, 76.1), turned to 90 degrees
- moved C9 16.3 mm to (82.8, 87.1)
- moved C10 16.2 mm to (82.8, 70.8)
- moved R26 16.0 mm to (89.5, 85.3), turned to -90 degrees
- moved R30 15.8 mm to (98.4, 85.3), turned to -90 degrees
- moved R27 14.0 mm to (91.7, 85.3), turned to -90 degrees
- moved R29 13.9 mm to (96.2, 85.3), turned to -90 degrees
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Connections:
- C18 pad 2: Net-(C18-Pad2) -> VIN
- D23 pad 2: unconnected-(D23-Pad2) -> +5V
- D24 pad 2: unconnected-(D24-Pad2) -> +5V
- F1 pad 1: Net-(C18-Pad2) -> VIN
- J15 pad 4: Net-(J15-Pad4) -> unconnected-(J15-Pad4)
- J15 pad 5: Net-(J15-Pad5) -> unconnected-(J15-Pad5)
- R1 pad 2: D3 -> D13
- R2 pad 2: D4 -> D12
- R29 pad 2: Net-(J15-Pad5) -> RD0
- R3 pad 2: D5 -> D11
- R30 pad 2: Net-(J15-Pad4) -> XD1
- U11 pad 1: unconnected-(U11-Pad1) -> GND
- U11 pad 2: unconnected-(U11-Pad2) -> GND
- U11 pad 3: unconnected-(U11-Pad3) -> GND
- U11 pad 4: unconnected-(U11-Pad4) -> GND
- U11 pad 7: unconnected-(U11-Pad7) -> GND
- U11 pad 8: unconnected-(U11-Pad8) -> Net-(U11-Pad8)
- U12 pad 1: unconnected-(U12-Pad1) -> RO
- U12 pad 2: unconnected-(U12-Pad2) -> Net-(Q7-Pad3)
- U12 pad 3: unconnected-(U12-Pad3) -> Net-(Q7-Pad3)
- U12 pad 4: unconnected-(U12-Pad4) -> GND
- U12 pad 5: unconnected-(U12-Pad5) -> GND
- U12 pad 6: unconnected-(U12-Pad6) -> Net-(U12-Pad6)
- U12 pad 7: unconnected-(U12-Pad7) -> Net-(U12-Pad7)
- U12 pad 8: unconnected-(U12-Pad8) -> Net-(R49-Pad1)
- U13 pad 1: unconnected-(U13-Pad1) -> Net-(U13-Pad1)
- U13 pad 2: unconnected-(U13-Pad2) -> Net-(U13-Pad2)
- U13 pad 3: unconnected-(U13-Pad3) -> Net-(BT2-Pad1)
- U13 pad 4: unconnected-(U13-Pad4) -> GND
- U13 pad 8: unconnected-(U13-Pad8) -> Net-(C23-Pad2)
- U14 pad 2: Net-(C18-Pad2) -> VIN
- U14 pad 3: unconnected-(U14-Pad3) -> GND
- U14 pad 4: Net-(U14-Pad4)_1 -> +5V
- U15 pad 1: unconnected-(U15-Pad1) -> Net-(U15-Pad2)
- U15 pad 2: unconnected-(U15-Pad2) -> Net-(U15-Pad2)
- U15 pad 3: unconnected-(U15-Pad3) -> Net-(C22-Pad2)
- U15 pad 4: unconnected-(U15-Pad4) -> GND
- U15 pad 5: unconnected-(U15-Pad5) -> Net-(U15-Pad2)
- U15 pad 6: unconnected-(U15-Pad6) -> Net-(U15-Pad6)
- U15 pad 7: unconnected-(U15-Pad7) -> Net-(U15-Pad7)
- U15 pad 8: unconnected-(U15-Pad8) -> VIN
- U16 pad 1: unconnected-(U16-Pad1) -> GND
- U16 pad 2: unconnected-(U16-Pad2) -> +3V3
- U16 pad 3: Net-(U14-Pad4)_1 -> +5V
- U2 pad 4: D13 -> A0
- U3 pad 4: A0 -> A1
- U4 pad 4: A1 -> A2
- U5 pad 4: A2 -> A3
- U6 pad 4: D12 -> D2
- U7 pad 4: D11 -> D3
- U8 pad 4: D10 -> D4
- U9 pad 4: D2 -> D5
- Y1 pad 1: X2 -> X1
- Y1 pad 2: X1 -> X2
Routing:
- net +5V: track 23.5 -> 129.2 mm, vias 0 -> 2
- net A6: track 14.8 -> 81.7 mm, vias 0 -> 4
- net A7: track 14.4 -> 80.0 mm, vias 0 -> 4
- net XD1: track 0.00 -> 58.4 mm, vias 0 -> 3
- net VIN: track 0.00 -> 43.8 mm, vias 0 -> 1
- net D9: track 0.00 -> 38.3 mm, vias 0 -> 2
- net D2: track 51.4 -> 15.8 mm, vias 2 -> 0
- net RD0: track 0.00 -> 34.2 mm, vias 0 -> 2
- net TXE: track 0.00 -> 33.3 mm, vias 0 -> 2
- net A4: track 3.50 -> 33.9 mm, vias 0 -> 3
- net +3V3: track 5.22 -> 34.6 mm
- net RO: track 0.00 -> 29.0 mm, vias 0 -> 2
- net D10: track 28.4 -> 0.00 mm
- net A5: track 2.91 -> 31.1 mm, vias 0 -> 3
- net RXE: track 0.00 -> 25.9 mm, vias 0 -> 2
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Other:
- outline, holes or cut-outs redrawn

Commit message: major update
Parts:
- moved R50 13.0 mm to (142.1, 102.0)
- moved R11 12.0 mm to (151.2, 64.6), turned to 90 degrees
- moved R52 4.06 mm to (155.0, 94.8)
- moved R53 1.97 mm to (150.9, 94.8), turned to -90 degrees
- moved R6 1.43 mm to (137.6, 68.5)
- moved R5 1.19 mm to (133.6, 68.1)
- moved D5 0.93 mm to (146.4, 64.5)
- moved Q6 0.75 mm to (154.4, 64.7)
- moved D11 0.63 mm to (140.8, 64.6)
- moved Je 0.54 mm to (143.2, 68.8)
- moved R10 0.50 mm to (129.6, 67.5)
- moved D12 0.44 mm to (157.7, 64.8)
- turned Q8 to -90 degrees
- turned Q9 to -90 degrees
- renumbered J18 to Je
Connections:
- Q8 pad 3: Net-(Q8-Pad3) -> A5
- Q9 pad 3: Net-(Q9-Pad3) -> A4
- R50 pad 2: Net-(Q8-Pad3) -> A5
- R51 pad 2: Net-(Q9-Pad3) -> A4
Routing:
- net Net-(D5-Pad1): track 0.00 -> 13.1 mm
- net Net-(Q6-Pad1): track 4.42 -> 16.7 mm
- net Net-(D11-Pad2): track 0.00 -> 11.4 mm
- net Net-(D4-Pad1): track 0.00 -> 4.73 mm
- net +3V3: track 34.6 -> 38.3 mm
- net Net-(D10-Pad2): track 8.20 -> 4.78 mm
- net D8: track 47.5 -> 44.1 mm
- net D7: track 42.5 -> 40.1 mm
- net Net-(Q5-Pad1): track 2.30 -> 3.95 mm
- net Net-(D11-Pad1): track 17.0 -> 16.3 mm

Commit message: Update #auto_saved_files#, Nano5-2022-04-10_203426.zip, and 8 more files...
Parts:
- moved R55 9.95 mm to (148.8, 95.0), turned to -90 degrees
- moved F1 9.71 mm to (153.8, 103.2)
- moved R54 4.24 mm to (152.9, 95.0), turned to -90 degrees
- moved R50 2.57 mm to (144.0, 103.6), turned to 0 degrees
- moved R51 1.86 mm to (144.0, 101.6)
- moved D22 1.71 mm to (152.1, 106.0)
- moved R52 0.31 mm to (155.0, 95.1)
- moved R53 0.23 mm to (150.9, 95.0)
- moved Q8 0.10 mm to (153.9, 99.1)

Commit message: update 2104
Parts:
- removed Je: Conn_01x05, Connector_PinHeader_2.54mm:PinHeader_1x05_P2.54mm_Vertical
- added D25: LED, LED_SMD:LED_0805_2012Metric, F.Cu at (126.0, 87.5)
- added J18: Conn_01x05, Connector_PinHeader_2.54mm:PinHeader_1x05_P2.54mm_Vertical, F.Cu at (143.9, 68.8)
- added R60: R, Resistor_SMD:R_0805_2012Metric, F.Cu at (136.0, 85.4)
- added SW2: SW_Push, Button_Switch_SMD:SW_SPST_B3U-1000P, F.Cu at (167.3, 68.7)
- added SW3: SW_Push, Button_Switch_SMD:SW_SPST_B3U-1000P, F.Cu at (78.5, 69.5)
- moved C18 2.61 mm to (142.8, 106.0), turned to 0 degrees
- moved C17 2.24 mm to (73.7, 70.1)
- moved R1 2.23 mm to (73.7, 67.9)
- moved K1 1.40 mm to (78.2, 59.9)
- moved K2 1.40 mm to (94.2, 59.9)
- moved K3 1.40 mm to (110.2, 59.9)
- moved K4 1.40 mm to (126.2, 59.9)
- moved K5 1.40 mm to (142.2, 59.9)
- moved K6 1.40 mm to (158.2, 59.9)
- moved R50 1.24 mm to (142.8, 103.7)
- moved R51 1.21 mm to (142.8, 101.5)
- moved C16 0.80 mm to (101.7, 78.0)
- moved R49 0.38 mm to (114.0, 70.9)
- moved JP4 0.31 mm to (114.3, 70.8)
- moved Q9 0.19 mm to (149.7, 98.9)
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Connections:
- J5 pad 1: unconnected-(J5-Pad1) -> OA
- J5 pad 2: unconnected-(J5-Pad2) -> OB
- J6 pad 1: unconnected-(J6-Pad1) -> GND
- J6 pad 2: unconnected-(J6-Pad2) -> AO
- J8 pad 1: Net-(J17-Pad1) -> Net-(J16-Pad1)
- J8 pad 3: Net-(J16-Pad1) -> Net-(J17-Pad1)
- R45 pad 2: unconnected-(R45-Pad2) -> OB
- R46 pad 2: unconnected-(R46-Pad2) -> OA
- R59 pad 2: unconnected-(R59-Pad2) -> AO
Routing:
- net OA: track 0.00 -> 92.7 mm, vias 0 -> 1
- net OB: track 0.00 -> 91.8 mm, vias 0 -> 1
- net AO: track 0.00 -> 87.6 mm, vias 0 -> 1
- net GND: track 5.83 -> 86.7 mm, vias 0 -> 12
- net A5: track 31.1 -> 95.0 mm, vias 3 -> 4
- net A4: track 33.9 -> 92.4 mm, vias 3 -> 4
- net +3V3: track 38.3 -> 83.4 mm, vias 0 -> 2
- net RST: track 5.06 -> 45.6 mm, vias 0 -> 2
- net +5V: track 129.2 -> 158.5 mm, vias 2 -> 5
- net RXE: track 25.9 -> 47.7 mm, vias 2 -> 3
- net TXE: track 33.3 -> 53.5 mm, vias 2 -> 3
- net Net-(J17-Pad1): track 7.27 -> 20.7 mm
- net ERST: track 6.26 -> 18.9 mm, vias 0 -> 1
- net ED2: track 3.27 -> 15.8 mm, vias 0 -> 2
- net Net-(D25-Pad2): track 0.00 -> 10.3 mm
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- added copper zone on B.Cu, net GND
- added copper zone on F.Cu, net GND

Commit message: fix update
Parts:
- added L1: L_Ferrite_Small, Inductor_SMD:L_1806_4516Metric_Pad1.45x1.90mm_HandSolder, F.Cu at (151.4, 105.2)
- F1: footprint Fuse:Fuse_0805_2012Metric -> Fuse:Fuse_1812_4532Metric
- moved F1 6.50 mm to (147.7, 105.4), turned to -90 degrees
- moved D22 2.74 mm to (154.7, 105.0), turned to -90 degrees
- moved BT2 0.61 mm to (136.5, 81.6)
Connections:
- F1 pad 2: Net-(D22-Pad1) -> Net-(F1-Pad2)
- J1 pad 1: unconnected-(J1-Pad1) -> Net-(K2-Pad1)
- J1 pad 2: unconnected-(J1-Pad2) -> Net-(K1-Pad3)
- J1 pad 3: unconnected-(J1-Pad3) -> Net-(K1-Pad1)
- J13 pad 1: unconnected-(J13-Pad1) -> +5V
- J13 pad 2: unconnected-(J13-Pad2) -> +3V3
- J13 pad 3: unconnected-(J13-Pad3) -> OB
- J13 pad 4: unconnected-(J13-Pad4) -> A4
- J13 pad 5: unconnected-(J13-Pad5) -> OA
- J13 pad 6: unconnected-(J13-Pad6) -> A5
- J13 pad 7: unconnected-(J13-Pad7) -> GND
- J13 pad 8: unconnected-(J13-Pad8) -> GND
- J14 pad 1: unconnected-(J14-Pad1) -> +5V
- J14 pad 2: unconnected-(J14-Pad2) -> +3V3
- J14 pad 3: unconnected-(J14-Pad3) -> OB
- J14 pad 4: unconnected-(J14-Pad4) -> A5
- J14 pad 5: unconnected-(J14-Pad5) -> OA
- J14 pad 6: unconnected-(J14-Pad6) -> A4
- J14 pad 7: unconnected-(J14-Pad7) -> GND
- J14 pad 8: unconnected-(J14-Pad8) -> GND
- J2 pad 1: unconnected-(J2-Pad1) -> Net-(J2-Pad1)
- J2 pad 2: unconnected-(J2-Pad2) -> Net-(J2-Pad2)
- J2 pad 3: unconnected-(J2-Pad3) -> Net-(K2-Pad3)
- J3 pad 1: unconnected-(J3-Pad1) -> Net-(K5-Pad1)
- J3 pad 2: unconnected-(J3-Pad2) -> Net-(K4-Pad3)
- J3 pad 3: unconnected-(J3-Pad3) -> Net-(K4-Pad1)
- J4 pad 1: unconnected-(J4-Pad1) -> Net-(J4-Pad1)
- J4 pad 2: unconnected-(J4-Pad2) -> Net-(K6-Pad1)
- J4 pad 3: unconnected-(J4-Pad3) -> Net-(K5-Pad3)
- K1 pad 1: unconnected-(K1-Pad1) -> Net-(K1-Pad1)
- K1 pad 3: unconnected-(K1-Pad3) -> Net-(K1-Pad3)
- K2 pad 1: unconnected-(K2-Pad1) -> Net-(K2-Pad1)
- K2 pad 3: unconnected-(K2-Pad3) -> Net-(K2-Pad3)
- K3 pad 1: unconnected-(K3-Pad1) -> Net-(J2-Pad2)
- K3 pad 3: unconnected-(K3-Pad3) -> Net-(J2-Pad1)
- K4 pad 1: unconnected-(K4-Pad1) -> Net-(K4-Pad1)
- K4 pad 3: unconnected-(K4-Pad3) -> Net-(K4-Pad3)
- K5 pad 1: unconnected-(K5-Pad1) -> Net-(K5-Pad1)
- K5 pad 3: unconnected-(K5-Pad3) -> Net-(K5-Pad3)
- K6 pad 1: unconnected-(K6-Pad1) -> Net-(K6-Pad1)
- K6 pad 3: unconnected-(K6-Pad3) -> Net-(J4-Pad1)
- U14 pad 1: unconnected-(U14-Pad1) -> GND
Routing:
- net OB: track 91.8 -> 282.6 mm, vias 1 -> 2
- net OA: track 92.7 -> 279.4 mm, vias 1 -> 2
- net A4: track 92.4 -> 233.7 mm, vias 4 -> 5
- net A5: track 95.0 -> 231.3 mm, vias 4 -> 5
- net +3V3: track 83.4 -> 194.2 mm, vias 2 -> 5
- net +5V: track 158.5 -> 258.8 mm, vias 5 -> 6
- net RD0: track 33.4 -> 82.2 mm
- net Net-(K6-Pad1): track 0.00 -> 45.6 mm
- net Net-(K5-Pad1): track 0.00 -> 38.0 mm
- net Net-(K5-Pad3): track 0.00 -> 37.7 mm
- net Net-(K4-Pad1): track 0.00 -> 34.4 mm
- net XD1: track 58.8 -> 92.9 mm
- net Net-(J4-Pad1): track 0.00 -> 32.2 mm
- net Net-(J2-Pad2): track 0.00 -> 28.0 mm
- net Net-(K1-Pad1): track 0.00 -> 25.9 mm
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- added copper zone on F.Cu, net +3V3

Commit message: ISP
Parts:
- added JP5: SolderJumper_3_Open, Jumper:SolderJumper-3_P1.3mm_Open_RoundedPad1.0x1.5mm, B.Cu at (79.8, 72.8)
- added JP6: SolderJumper_3_Open, Jumper:SolderJumper-3_P1.3mm_Open_RoundedPad1.0x1.5mm, B.Cu at (76.6, 72.8)
- added JP7: SolderJumper_3_Open, Jumper:SolderJumper-3_P1.3mm_Open_RoundedPad1.0x1.5mm, B.Cu at (73.4, 72.8)
Connections:
- C17 pad 1: unconnected-(C17-Pad1) -> DTR
- J15 pad 1: unconnected-(J15-Pad1) -> JD12
- J15 pad 2: unconnected-(J15-Pad2) -> +5V
- J15 pad 3: unconnected-(J15-Pad3) -> JD13
- J15 pad 4: unconnected-(J15-Pad4) -> D11
- J15 pad 5: unconnected-(J15-Pad5) -> JRST
- J15 pad 6: unconnected-(J15-Pad6) -> GND
Routing:
- net D11: track 11.3 -> 47.8 mm, vias 0 -> 1
- net +5V: track 258.8 -> 279.9 mm
- net D12: track 4.05 -> 19.4 mm, vias 0 -> 1
- net JD13: track 0.00 -> 8.09 mm, vias 0 -> 1
- net JD12: track 0.00 -> 5.11 mm, vias 0 -> 1
- net XD1: track 92.9 -> 97.7 mm
- net D13: track 19.4 -> 23.5 mm, vias 0 -> 1
- net Net-(J3-Pad1): track 38.0 -> 39.9 mm
- net RD0: track 82.2 -> 82.9 mm
- net Net-(J2-Pad1): track 15.1 -> 15.7 mm

Commit message: fix track
Parts:
- added JP8: Jumper_2_Bridged, Jumper:SolderJumper-2_P1.3mm_Bridged2Bar_RoundedPad1.0x1.5mm, B.Cu at (72.0, 63.5)
- added TP1: TestPoint, TestPoint:TestPoint_Pad_D1.0mm, F.Cu at (93.2, 67.6)
- JP2, JP3, JP4: footprint Jumper:SolderJumper-2_P1.3mm_Bridged_RoundedPad1.0x1.5mm -> Jumper:SolderJumper-2_P1.3mm_Open_RoundedPad1.0x1.5mm
Connections:
- D1 pad 1: Net-(D1-Pad1) -> +5P
- D2 pad 1: Net-(D2-Pad1) -> +5P
- D3 pad 1: Net-(D3-Pad1) -> +5P
- D4 pad 1: Net-(D4-Pad1) -> +5P
- D5 pad 1: Net-(D5-Pad1) -> +5P
- D6 pad 1: Net-(D6-Pad1) -> +5P
- J12 pad 2: unconnected-(J12-Pad2) -> GND
- J7 pad 1: unconnected-(J7-Pad1) -> +5V
- J7 pad 2: unconnected-(J7-Pad2) -> GND
- K1 pad 2: Net-(D1-Pad1) -> +5P
- K2 pad 2: Net-(D2-Pad1) -> +5P
- K3 pad 2: Net-(D3-Pad1) -> +5P
- K4 pad 2: Net-(D4-Pad1) -> +5P
- K5 pad 2: Net-(D5-Pad1) -> +5P
- K6 pad 2: Net-(D6-Pad1) -> +5P
- R10 pad 2: Net-(D4-Pad1) -> +5P
- R11 pad 2: Net-(D5-Pad1) -> +5P
- R12 pad 2: Net-(D6-Pad1) -> +5P
- R7 pad 2: Net-(D1-Pad1) -> +5P
- R8 pad 2: Net-(D2-Pad1) -> +5P
- R9 pad 2: Net-(D3-Pad1) -> +5P
Routing:
- net +5P: track 0.00 -> 191.6 mm
- net +5V: track 279.9 -> 328.4 mm, vias 6 -> 7
- net JRST: track 0.00 -> 14.8 mm, vias 0 -> 1
- net Net-(D3-Pad1): track 12.5 -> 0.00 mm
- net Net-(D2-Pad1): track 12.2 -> 0.00 mm
- net Net-(D4-Pad1): track 12.0 -> 0.00 mm
- net Net-(D1-Pad1): track 10.5 -> 0.00 mm
- net Net-(D6-Pad1): track 10.2 -> 0.00 mm
- net Net-(D5-Pad1): track 10.1 -> 0.00 mm
- net DTR: track 0.00 -> 9.47 mm, vias 0 -> 1
- net D10: track 0.00 -> 4.49 mm, vias 0 -> 2
- net GND: track 92.0 -> 89.4 mm

Commit message: update annote
Parts:
- added FID1: Fiducial, Fiducial:Fiducial_1.5mm_Mask3mm, F.Cu at (166.9, 110.5)
- added FID2: Fiducial, Fiducial:Fiducial_1.5mm_Mask3mm, F.Cu at (73.4, 110.7)
- added FID3: Fiducial, Fiducial:Fiducial_1.5mm_Mask3mm, F.Cu at (73.4, 39.4)
- added FID4: Fiducial, Fiducial:Fiducial_1.5mm_Mask3mm, F.Cu at (164.2, 51.9)
- added JP9: Jumper_2_Bridged, Jumper:SolderJumper-2_P1.3mm_Bridged_RoundedPad1.0x1.5mm, B.Cu at (154.9, 85.7)
- added Re1: R, Resistor_THT:R_Axial_DIN0207_L6.3mm_D2.5mm_P10.16mm_Horizontal, F.Cu at (168.1, 45.1)
- H1, H2, H3, H4: value MountingHole -> MountingHole_Pad; footprint MountingHole:MountingHole_3.2mm_M3 -> MountingHole:MountingHole_3.2mm_M3_Pad_Via
- moved R12 0.38 mm to (167.9, 64.7)
Connections:
- J7 pad 1: +5V -> GND
- J7 pad 2: GND -> +5V
- J8 pad 2: unconnected-(J8-Pad2) -> GND
- Q10 pad 2: RXE -> Net-(Q10-Pad2)
- R58 pad 2: RXE -> Net-(Q10-Pad2)
Routing:
- net Net-(Q10-Pad2): track 0.00 -> 21.2 mm, vias 0 -> 1
- net RXE: track 46.4 -> 26.9 mm, vias 3 -> 2
- net Net-(Re1-Pad1): track 0.00 -> 12.0 mm
- net GND: track 89.4 -> 100.7 mm
- net TXE: track 52.4 -> 56.0 mm
- net +3V3: track 194.2 -> 192.6 mm
- net XD1: track 97.7 -> 96.3 mm
- net Net-(D1-Pad2): track 15.1 -> 14.0 mm
- net Net-(D2-Pad2): track 14.9 -> 14.0 mm
- net A5: track 231.3 -> 230.4 mm
- net VIN: track 63.5 -> 62.8 mm
- net Net-(U13-Pad2): track 9.50 -> 8.81 mm
- net Net-(J16-Pad1): track 18.3 -> 17.7 mm
- net +5P: track 191.6 -> 191.1 mm
Other:
- board text added: "+ INPUT -"
- board text added: "+ OUTPUT -"
- board text added: "2=3V3 1=5V 4=A4 3=OB 6=A5 5=OA 8=GND 7=GND"
- board text added: "485"
- board text added: "5V+"
- board text added: "A"
- board text added: "A B"
- board text added: "AIN0"
- board text added: "AIN1"
- board text added: "AIN_MODE"
- board text added: "BY: RJLABS"
- board text added: "COMMON"
- board text added: "CR2302"
- board text added: "D11"
- board text added: "DEV0"
- board text added: "DTR"
- board text added: "DTR.RX.TX"
- board text added: "EEPROM"
- board text added: "ESP"
- board text added: "ESP PROG"
- board text added: "GIN"
- board text added: "GND"
- board text added: "GND AO"
- board text added: "Gnd"
- board text added: "I.0 RST TX RX GND"
- board text added: "J13/J14 PINOUT:"
- board text added: "MODBUS"
- board text added: "NANO5_PLC by:"
- board text added: "PG"
- board text added: "R6 C R5 C R4 C R3 C R2 C R1 C"
- board text added: "RJLabs Innovation"
- board text added: "RST.D12.D13"
- board text added: "RTC"
- board text added: "RX"
- board text added: "S8 S7 S6 S5 S4 S3 S2 S1"
- board text added: "TX"
- board text added: "V"
- board text added: "V.2.0"
- board text added: "VIN"
- board text added: "VIN RELAY"
