File: HW/frame/frame.kicad_pcb (KiCad board)
At the start: 2 copper layers, 100 x 90 mm, 4 parts

Commit message: phase 1
Parts:
- added D1: SM4007, Diode_SMD:D_MELF, F.Cu at (80.5, 65.1)
- added D10: LED, LED_SMD:LED_0805_2012Metric, F.Cu at (104.8, 92.2)
- added D11: LED, LED_SMD:LED_0805_2012Metric, F.Cu at (104.8, 95.2)
- added D12: LED, LED_SMD:LED_0805_2012Metric, F.Cu at (109.3, 92.2)
- added D2: SM4007, Diode_SMD:D_MELF, F.Cu at (96.5, 65.1)
- added D3: SM4007, Diode_SMD:D_MELF, F.Cu at (112.4, 65.1)
- added D4: SM4007, Diode_SMD:D_MELF, F.Cu at (128.5, 65.2)
- added D5: SM4007, Diode_SMD:D_MELF, F.Cu at (144.6, 65.2)
- added D6: SM4007, Diode_SMD:D_MELF, F.Cu at (160.6, 65.0)
- added D7: LED, LED_SMD:LED_0805_2012Metric, F.Cu at (79.0, 68.3)
- added D8: LED, LED_SMD:LED_0805_2012Metric, F.Cu at (113.7, 92.2)
- added D9: LED, LED_SMD:LED_0805_2012Metric, F.Cu at (104.8, 98.2)
- added J1: Screw_Terminal_01x03, TerminalBlock_Phoenix:TerminalBlock_Phoenix_MKDS-1,5-3-5.08_1x03_P5.08mm_Horizontal, F.Cu at (91.5, 35.4)
- added J2: Screw_Terminal_01x03, TerminalBlock_Phoenix:TerminalBlock_Phoenix_MKDS-1,5-3-5.08_1x03_P5.08mm_Horizontal, F.Cu at (107.0, 35.4)
- added J3: Screw_Terminal_01x03, TerminalBlock_Phoenix:TerminalBlock_Phoenix_MKDS-1,5-3-5.08_1x03_P5.08mm_Horizontal, F.Cu at (122.5, 35.4)
- added J4: Screw_Terminal_01x03, TerminalBlock_Phoenix:TerminalBlock_Phoenix_MKDS-1,5-3-5.08_1x03_P5.08mm_Horizontal, F.Cu at (138.1, 35.4)
- added J5: Screw_Terminal_01x03, TerminalBlock_Phoenix:TerminalBlock_Phoenix_MKDS-1,5-3-5.08_1x03_P5.08mm_Horizontal, F.Cu at (205.7, 40.7)
- added J6: Screw_Terminal_01x04, TerminalBlock_Phoenix:TerminalBlock_Phoenix_MKDS-1,5-4-5.08_1x04_P5.08mm_Horizontal, F.Cu at (158.6, 35.4)
- added K1: SANYOU_SRD_Form_C, Relay_THT:Relay_SPDT_SANYOU_SRD_Series_Form_C, F.Cu at (79.7, 60.0)
- added K2: SANYOU_SRD_Form_C, Relay_THT:Relay_SPDT_SANYOU_SRD_Series_Form_C, F.Cu at (95.7, 60.0)
- added K3: SANYOU_SRD_Form_C, Relay_THT:Relay_SPDT_SANYOU_SRD_Series_Form_C, F.Cu at (111.7, 60.0)
- added K4: SANYOU_SRD_Form_C, Relay_THT:Relay_SPDT_SANYOU_SRD_Series_Form_C, F.Cu at (127.7, 60.0)
- added K5: SANYOU_SRD_Form_C, Relay_THT:Relay_SPDT_SANYOU_SRD_Series_Form_C, F.Cu at (143.7, 60.0)
- added K6: SANYOU_SRD_Form_C, Relay_THT:Relay_SPDT_SANYOU_SRD_Series_Form_C, F.Cu at (159.7, 60.0)
- added Q1: MMBT3904, Package_TO_SOT_SMD:SOT-23, F.Cu at (73.7, 64.8)
- added Q2: MMBT3904, Package_TO_SOT_SMD:SOT-23, F.Cu at (89.7, 64.8)
- added Q3: MMBT3904, Package_TO_SOT_SMD:SOT-23, F.Cu at (105.7, 64.8)
- added Q4: MMBT3904, Package_TO_SOT_SMD:SOT-23, F.Cu at (121.7, 64.9)
- added Q5: MMBT3904, Package_TO_SOT_SMD:SOT-23, F.Cu at (137.7, 64.8)
- added Q6: MMBT3904, Package_TO_SOT_SMD:SOT-23, F.Cu at (153.7, 64.8)
- added R1: R, Resistor_SMD:R_0805_2012Metric, F.Cu at (73.6, 68.3)
- added R10: R, Resistor_SMD:R_0805_2012Metric, F.Cu at (118.1, 95.1)
- added R11: R, Resistor_SMD:R_0805_2012Metric, F.Cu at (113.6, 98.2)
- added R12: R, Resistor_SMD:R_0805_2012Metric, F.Cu at (118.0, 98.1)
- added R2: R, Resistor_SMD:R_0805_2012Metric, F.Cu at (89.7, 69.0)
- added R3: R, Resistor_SMD:R_0805_2012Metric, F.Cu at (105.6, 69.3)
- added R4: R, Resistor_SMD:R_0805_2012Metric, F.Cu at (121.5, 69.1)
- added R5: R, Resistor_SMD:R_0805_2012Metric, F.Cu at (137.7, 69.1)
- added R6: R, Resistor_SMD:R_0805_2012Metric, F.Cu at (153.7, 69.3)
- added R7: R, Resistor_SMD:R_0805_2012Metric, F.Cu at (83.3, 68.3)
- added R8: R, Resistor_SMD:R_0805_2012Metric, F.Cu at (109.2, 98.2)
- added R9: R, Resistor_SMD:R_0805_2012Metric, F.Cu at (118.1, 92.1)

Commit message: add mod 1
Parts:
- added J10: Screw_Terminal_01x03, TerminalBlock_Phoenix:TerminalBlock_Phoenix_MKDS-1,5-3-5.08_1x03_P5.08mm_Horizontal, F.Cu at (97.2, 114.3)
- added J11: Screw_Terminal_01x03, TerminalBlock_Phoenix:TerminalBlock_Phoenix_MKDS-1,5-3-5.08_1x03_P5.08mm_Horizontal, F.Cu at (81.7, 114.3)
- added J12: Screw_Terminal_01x02, TerminalBlock_Phoenix:TerminalBlock_Phoenix_MKDS-1,5-2_1x02_P5.00mm_Horizontal, F.Cu at (153.9, 114.3)
- added J7: Screw_Terminal_01x02, TerminalBlock_Phoenix:TerminalBlock_Phoenix_MKDS-1,5-2_1x02_P5.00mm_Horizontal, F.Cu at (143.7, 114.3)
- added J8: Screw_Terminal_01x03, TerminalBlock_Phoenix:TerminalBlock_Phoenix_MKDS-1,5-3-5.08_1x03_P5.08mm_Horizontal, F.Cu at (128.2, 114.3)
- added J9: Screw_Terminal_01x03, TerminalBlock_Phoenix:TerminalBlock_Phoenix_MKDS-1,5-3-5.08_1x03_P5.08mm_Horizontal, F.Cu at (112.7, 114.3)
- J5: value Screw_Terminal_01x03 -> Screw_Terminal_01x02; footprint TerminalBlock_Phoenix:TerminalBlock_Phoenix_MKDS-1,5-3-5.08_1x03_P5.08mm_Horizontal -> TerminalBlock_Phoenix:TerminalBlock_Phoenix_MKDS-1,5-2_1x02_P5.00mm_Horizontal
- J6: value Screw_Terminal_01x04 -> Screw_Terminal_01x02; footprint TerminalBlock_Phoenix:TerminalBlock_Phoenix_MKDS-1,5-4-5.08_1x04_P5.08mm_Horizontal -> TerminalBlock_Phoenix:TerminalBlock_Phoenix_MKDS-1,5-2_1x02_P5.00mm_Horizontal
- moved J5 57.6 mm to (148.3, 35.4)
- moved R12 55.6 mm to (164.8, 68.0)
- moved D12 55.2 mm to (157.2, 64.8), turned to -90 degrees
- moved D11 47.6 mm to (141.4, 64.8), turned to -90 degrees
- moved R11 46.3 mm to (148.8, 68.0)
- moved D8 34.2 mm to (93.3, 64.8), turned to -90 degrees
- moved D10 34.1 mm to (125.2, 64.8), turned to -90 degrees
- moved D9 33.8 mm to (109.5, 64.8), turned to -90 degrees
- moved R8 31.3 mm to (100.8, 68.1)
- moved R10 30.8 mm to (132.8, 68.0)
- moved R9 24.1 mm to (116.8, 68.1)
- moved D7 3.91 mm to (77.2, 64.8), turned to -90 degrees
- moved D3 2.93 mm to (115.3, 64.6)
- moved D1 2.87 mm to (83.3, 64.6)
- moved D4 2.87 mm to (131.3, 64.6)
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Routing:
- net Net-(D10-Pad1): track 0.00 -> 17.2 mm
- net Net-(D3-Pad2): track 0.00 -> 17.1 mm
- net Net-(D12-Pad1): track 0.00 -> 17.1 mm
- net Net-(D1-Pad2): track 0.00 -> 17.0 mm
- net Net-(D11-Pad1): track 0.00 -> 17.0 mm
- net Net-(D2-Pad2): track 0.00 -> 17.0 mm
- net Net-(D2-Pad1): track 0.00 -> 10.0 mm
- net Net-(D3-Pad1): track 0.00 -> 10.0 mm
- net Net-(D4-Pad1): track 0.00 -> 10.0 mm
- net Net-(D1-Pad1): track 0.00 -> 10.0 mm
- net Net-(D5-Pad1): track 0.00 -> 9.98 mm
- net Net-(D6-Pad1): track 0.00 -> 9.95 mm
- net Net-(D8-Pad2): track 0.00 -> 8.36 mm
- net Net-(D10-Pad2): track 0.00 -> 8.20 mm
- net Net-(D7-Pad2): track 0.00 -> 8.12 mm
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